File: SingleBoard/SingleBoard.kicad_sch (KiCad schematic)
At the start: 0 parts

Commit message: Created Pcb
Parts:
- added D1, D10, D11, D12, D13, D14, D15, D16, D17, D18, D19, D2, D3, D4, D5, D6, D7, D8, D9, DR1: 1N4148, Diode_THT:D_DO-35_SOD27_P7.62mm_Horizontal, symbol Diode:1N4148
- added SW1, SW10, SW11, SW12, SW13, SW14, SW15, SW16, SW17, SW18, SW19, SW2, SW3, SW4, SW5, SW6, SW7, SW8, SW9: SW_Push_45deg, Button_Switch_Keyboard:SW_Cherry_MX_1.00u_PCB, symbol Switch:SW_Push_45deg
- added SWR1: RotaryEncoder_Switch, Rotary_Encoder:RotaryEncoder_Alps_EC11E-Switch_Vertical_H20mm, symbol Device:RotaryEncoder_Switch
- added U2: Seeed Studio XIAO RP2040, footprintshack:XIAO-Generic-Hybrid-14P-2.54-21X17.8MM, symbol Seeed_Studio_XIAO_Series:Seeed Studio XIAO SAMD21
Connections:
- new net: D12.2 (A), SW12.2
- new net: D16.2 (A), SW16.2
- new net: D5.2 (A), SW5.2
- new net: D2.2 (A), SW2.2
- new net: D3.2 (A), SW3.2
- new net: D4.2 (A), SW4.2
- new net: D7.2 (A), SW7.2
- new net: D13.2 (A), SW13.2
- new net: D15.2 (A), SW15.2
- new net: D9.2 (A), SW9.2
- new net: D8.2 (A), SW8.2
- new net: D14.2 (A), SW14.2
- new net: D10.2 (A), SW10.2
- new net: D18.2 (A), SW18.2
- new net: D17.2 (A), SW17.2
- new net: D1.2 (A), SW1.2
- new net: D6.2 (A), SW6.2
- new net: D11.2 (A), SW11.2
- new net: D19.2 (A), SW19.2
- new net Column0: SW1.1, SW2.1, SW3.1, SW4.1, SWR1.S1, U2.1 (PA02_A0_D0)
- new net Column1: SW5.1, SW6.1, SW7.1, SW8.1, SW9.1, U2.2 (PA4_A1_D1)
- new net Column2: SW10.1, SW11.1, SW12.1, SW13.1, SW14.1, U2.3 (PA10_A2_D2)
- new net Column3: SW15.1, SW16.1, SW17.1, SW18.1, SW19.1, U2.4 (PA11_A3_D3)
- new net EC11A: SWR1.A, U2.6 (PA9_A5_D5_SCL)
- new net EC11B: SWR1.B, U2.5 (PA8_A4_D4_SDA)
- new net EC11SWA: DR1.2 (A), SWR1.S2
- new net GND: SWR1.C, U2.13 (GND)
- new net ROW0: D1.1 (K), D10.1 (K), D15.1 (K), D5.1 (K), U2.8 (PB09_A7_D7_RX)
- new net ROW1: D11.1 (K), D16.1 (K), D2.1 (K), D6.1 (K), U2.9 (PA7_A8_D8_SCK)
- new net ROW2: D12.1 (K), D17.1 (K), D3.1 (K), D7.1 (K), U2.10 (PA5_A9_D9_MISO)
- new net ROW3: D13.1 (K), D18.1 (K), D4.1 (K), D8.1 (K), U2.11 (PA6_A10_D10_MOSI)
- new net ROW4: D14.1 (K), D19.1 (K), D9.1 (K), DR1.1 (K), U2.7 (PB08_A6_D6_TX)
- new net VCC: U2.14 (5V)
Other:
- note added: "Rotary Encoder"
